File: hardware/pcbs/board/board.kicad_pcb (KiCad board)
At the start: 2 copper layers, 153.4 x 104.5 mm, 72 parts, among them K00 Key, K01 Key, K02 Key, K03 Key, K10 Key, K11 Key, K12 Key, K13 Key, K20 Key, K21 Key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

Commit message: updates to pcb and case
Parts:
- Battery1, BatteryJmp1, Reset1: moved to B.Cu
- moved Battery1 23.0 mm to (135.8, 112.1), turned to -90 degrees
- moved BatteryJmp1 14.9 mm to (150.6, 132.1), turned to -90 degrees
- moved D00 14.4 mm to (96.5, 119.4), turned to -90 degrees
- moved D01 13.7 mm to (96.5, 100.3), turned to -90 degrees
- moved D21 12.0 mm to (116.8, 85.1), turned to -90 degrees
- moved D20 12.0 mm to (116.8, 105.4), turned to -90 degrees
- moved D02 11.4 mm to (96.5, 80.0), turned to 90 degrees
- moved D30 10.9 mm to (154.9, 97.8), turned to -90 degrees
- moved D03 10.2 mm to (96.5, 64.8), turned to 90 degrees
- moved D31 9.16 mm to (154.9, 78.7), turned to -90 degrees
- moved Reset1 6.50 mm to (204.6, 134.6), turned to 180 degrees
- moved LevelShift1 1.75 mm to (199.9, 106.8)
- moved C1 1.03 mm to (195.6, 108.1)
- turned K00 to -90 degrees
- turned K01 to -90 degrees
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Routing:
- net Net-(Battery1-Pad1): track 45.0 -> 15.8 mm
- net Col2: track 119.4 -> 136.3 mm
- net Col0: track 161.2 -> 170.6 mm
- net Row1: track 226.9 -> 219.2 mm
- net Row2: track 193.5 -> 185.9 mm
- net Col3: track 103.5 -> 111.0 mm
- net Row3: track 207.0 -> 199.5 mm
- net Row0: track 161.0 -> 156.1 mm
- net Col1: track 140.2 -> 144.7 mm
- net Net-(D00-Pad2): track 5.87 -> 9.74 mm
- net Net-(D02-Pad2): track 9.55 -> 6.00 mm
- net Net-(D31-Pad2): track 8.32 -> 5.45 mm
- net Col5: track 113.1 -> 110.3 mm
- net Net-(D01-Pad2): track 7.87 -> 10.2 mm
- net Net-(D20-Pad2): track 6.96 -> 9.23 mm
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Other:
- board size 153.4 x 104.5 mm -> 146.6 x 105.2 mm
- board text added: "Light Barrier"

Commit message: pcb updates
Parts:
- removed the Battery1 at (135.8, 112.1)
- removed BoostConverter1: MP9361, Package_TO_SOT_SMD:SOT-23-6
- removed C3: 0.47uF, Capacitor_SMD:C_0805_2012Metric_Pad1.18x1.45mm_HandSolder
- removed LevelShift1: SN74LVC1T45DRL, Package_TO_SOT_SMD:SOT-563
- removed the Nice!NanoV2 at (188.0, 143.5)
- removed the Nice!NanoV2 at (165.1, 143.5)
- added Battery1: Battery_Cell, SVastaCustomParts:BatteryHolder_Keystone_1088_1xAA, F.Cu at (135.9, 106.7)
- added Battery1: Battery_Cell, SVastaCustomParts:BatteryHolder_Keystone_1088_1xAA, B.Cu at (135.9, 106.7)
- added Boost1: XC9142, SVastaCustomParts:SOT-25-5, F.Cu at (197.3, 99.6)
- added G***: LOGO, SVastaCustomParts:wing_it, F.Cu at (110.5, 126.4)
- added G***: LOGO, SVastaCustomParts:wing_it, B.Cu at (111.1, 130.8)
- added L1: 4.7uH, Inductor_SMD:L_0805_2012Metric_Pad1.15x1.40mm_HandSolder, F.Cu at (195.1, 95.8)
- added LvlShft1: TXB0101, Package_TO_SOT_SMD:SOT-23-6_Handsoldering, F.Cu at (200.7, 108.6)
- added Nice!NanoV2: Nice!Nano V2 Socket, SVastaCustomParts:Nice!NanoSocket_Reversible, F.Cu at (176.5, 128.9)
- C1, C2: value 2.2uF -> 10uF
- moved D60 30.5 mm to (198.7, 142.9), turned to 0 degrees
- moved D61 26.6 mm to (198.8, 139.1), turned to 0 degrees
- moved C1 7.11 mm to (193.4, 101.3), turned to 120 degrees
- moved C2 5.92 mm to (199.5, 103.5), turned to 30 degrees
- moved Reset1 4.91 mm to (202.0, 130.5)
Connections:
- C1 pad 1: /Peripheral 3.3V Supply -> GND
- C1 pad 2: Net-(BoostConverter1-Pad5) -> /Peripheral 3.3V Supply
- C2 pad 1: Net-(BoostConverter1-Pad1) -> GND
Routing:
- net GND: track 3.17 -> 55.0 mm, vias 15 -> 33
- net Col4: track 86.1 -> 127.9 mm, vias 0 -> 3
- net Row0: track 156.1 -> 194.8 mm, vias 0 -> 3
- net Col5: track 110.3 -> 135.6 mm, vias 0 -> 2
- net LED Control: track 64.6 -> 40.3 mm, vias 0 -> 2
- net Col6: track 49.4 -> 73.6 mm, vias 0 -> 1
- net Col2: track 136.3 -> 158.4 mm, vias 0 -> 2
- net Bat+: track 34.6 -> 55.9 mm, vias 0 -> 2
- net Col3: track 111.0 -> 132.0 mm, vias 0 -> 3
- net Row2: track 185.9 -> 200.5 mm, vias 2 -> 1
- net Net-(Nice!NanoV2-Pad22): track 33.5 -> 47.5 mm, vias 0 -> 2
- net /Peripheral 3.3V Supply: track 54.1 -> 67.7 mm, vias 0 -> 1
- net Row1: track 219.2 -> 205.8 mm, vias 2 -> 3
- net Col0: track 170.6 -> 160.6 mm, vias 0 -> 1
- net Row3: track 199.5 -> 209.3 mm
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Other:
- outline, holes or cut-outs redrawn
- board text added: "Designed by Sam Vasta ©2022"
